File: esp32wroverbreakout.kicad_pcb (KiCad board)
At the start: 2 copper layers, 34.3 x 53.3 mm, 27 parts, among them J2 hdr1, J3 hdr2, U1 TPS82140, U2 TPS3839DBZ, U3 ESP32-WROVER

Commit message: Add files via upload
Parts:
- removed PGM: PGM, ESP-WROOM-32-Breakout:DTSM-3
- removed PGM/DBG: PGM/DBG, Connector_PinSocket_2.54mm:PinSocket_1x04_P2.54mm_Vertical
- removed RST: RST, ESP-WROOM-32-Breakout:DTSM-3
- removed VIN: VIN, Connector_PinSocket_2.54mm:PinSocket_1x03_P2.54mm_Vertical
- added J1: VIN, Connector_PinSocket_2.54mm:PinSocket_1x03_P2.54mm_Vertical, F.Cu at (106.7, 105.3)
- added J4: PGM/DBG, Connector_PinSocket_2.54mm:PinSocket_1x04_P2.54mm_Vertical, F.Cu at (128.2, 105.0)
- added S1: RST, ESP-WROOM-32-Breakout:DTSM-3, F.Cu at (117.4, 103.5)
- added S2: PGM, ESP-WROOM-32-Breakout:DTSM-3, F.Cu at (133.6, 103.5)
- moved R2 2.21 mm to (119.2, 90.9)
- moved U2 1.01 mm to (119.4, 93.7)
- moved C6 0.91 mm to (122.1, 93.3)
Connections:
- C5 pad 1: Net-(C3-Pad1) -> +3V3
Routing:
- net Net-(C3-Pad1): track 23.1 -> 16.1 mm
- net RST: track 48.4 -> 46.4 mm
- net +3V3: track 3.67 -> 2.25 mm, vias 14 -> 18
- net Net-(J4-Pad4): track 8.13 -> 6.76 mm
- net IO13: track 14.7 -> 15.8 mm
- net GND: track 1.17 -> 0.42 mm
- net TXD0: track 42.5 -> 43.2 mm
Other:
- board text added: "E"
- board text added: "G"
- board text added: "PGM"
- board text added: "RST"
- board text added: "V"
- board text removed: "EN"
- board text removed: "VB"
