File: esp32wroverbreakout.sch (KiCad schematic (older format))
At the start: 27 parts, among them J1 VIN, J2 hdr1, J3 hdr2, J4 PGM/DBG, U1 TPS82140, U2 TPS3839DBZ, U3 ESP32-WROVER

Commit message: Add files via upload
Connections:
- net +3V3: now also C5.1
- net at C3.1, C4.1, JP1.3 (B)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: no longer C5.1
Other:
- moved on the sheet: C5
Changed lines of the file:
@@
 $EndComp
 Connection ~ 3850 4750
-Wire Wire Line
-	3850 4750 4250 4750
 $Comp
 L Device:C C5
 U 1 1 5C4A1E90
-P 4250 4900
-F 0 "C5" H 4365 4946 50  0000 L CNN
-F 1 "220u" H 4365 4855 50  0000 L CNN
-F 2 "Capacitor_Tantalum_SMD:CP_EIA-6032-28_Kemet-C" H 4288 4750 50  0001 C CNN
-F 3 "~" H 4250 4900 50  0001 C CNN
-	1    4250 4900
-	1    0    0    -1
-$EndComp
-Connection ~ 4250 4750
-Wire Wire Line
-	4250 4750 4600 4750
+P 5000 2200
+F 0 "C5" H 5115 2246 50  0000 L CNN
+F 1 "220u" H 5115 2155 50  0000 L CNN
+F 2 "Capacitor_Tantalum_SMD:CP_EIA-6032-28_Kemet-C" H 5038 2050 50  0001 C CNN
+F 3 "~" H 5000 2200 50  0001 C CNN
+	1    5000 2200
+	1    0    0    -1
+$EndComp
 $Comp
 L Device:R R4
@@
 L power:GND #PWR08
 U 1 1 5C4A3A2A
-P 4050 5050
-F 0 "#PWR08" H 4050 4800 50  0001 C CNN
-F 1 "GND" H 4055 4877 50  0000 C CNN
-F 2 "" H 4050 5050 50  0001 C CNN
-F 3 "" H 4050 5050 50  0001 C CNN
-	1    4050 5050
-	1    0    0    -1
-$EndComp
-Wire Wire Line
-	3850 5050 4050 5050
-Wire Wire Line
-	4050 5050 4250 5050
-Connection ~ 4050 5050
+P 3850 5050
+F 0 "#PWR08" H 3850 4800 50  0001 C CNN
+F 1 "GND" H 3855 4877 50  0000 C CNN
+F 2 "" H 3850 5050 50  0001 C CNN
+F 3 "" H 3850 5050 50  0001 C CNN
+	1    3850 5050
+	1    0    0    -1
+$EndComp
 $Comp
 L Device:C C1
@@
 Wire Wire Line
 	5350 2050 5700 2050
+Wire Wire Line
+	3850 4750 4600 4750
+Wire Wire Line
+	5000 2350 5350 2350
+Connection ~ 5350 2350
+Wire Wire Line
+	5000 2050 5350 2050
+Connection ~ 5350 2050
 $EndSCHEMATC
